File: WiFi DAC.sch (EAGLE design)
At the start: 11 parts

Commit message: Meer op z'n plek
Parts:
- added C1, C11, C2, C3, C4: 100nF, rcl:C-EUC0603
- added C10, C9: 47uF, rcl:CPOL-EUSANYO_SMD_A5
- added C5, C6: 2.2uF, rcl:C-EUC0603
- added C7, C8: 2200pF, rcl:C-EUC0603
- added R10, R11, R9: 47k, rcl:R-EU_R0603
- added R7, R8: 470, rcl:R-EU_R0603
- R1, R2, R3, R4, R5, R6: value (none) -> 33
Connections:
- new net +3V3: C1.1, C10.+, C11.1, C9.+, MDL1.VCC, U$2.AVDD, U$2.CPVDD, U$2.DVDD, U$2.XSMT, U1.OUT, U1.OUT@1
- new net +5V: U$1.5V0@1, U$1.5V0@2, U1.IN
- new net N$17: C2.1, U$2.LDOO
- new net N$18: C3.2, C5.2, U$2.CAPM
- new net N$19: C3.1, C5.1, U$2.CAPP
- new net N$20: C4.1, C6.1, U$2.VNEG
- new net N$21: C7.2, JP1.LEFT, R7.2
- new net N$22: C8.2, JP1.RIGHT, R8.2
- new net N$23: R7.1, U$2.OUTL
- new net N$24: R8.1, U$2.OUTR
- new net N$25: R9.2, U$2.DEMP
- new net N$26: R10.2, U$2.FLT
- new net N$27: R11.2, U$2.FMT
- net GND: now also C1.2, C10.-, C11.2, C2.2, C4.2, C6.2, C7.1, C8.1, C9.-, JP1.SLEEVE, MDL1.GND, R10.1, R11.1, R9.1, U1.ADJ
Other:
- moved on the sheet: JP1
