File: WiFi DAC2.brd (EAGLE design)
At the start: 65 x 30 mm, 29 parts

Commit message: test
jup
Routing:
- net N$3: track 3.60 -> 3.06 mm
Other:
- board text added: "Rev 1, 8-6-2016"
- board text added: "Sebastius"
- board text added: "WiFi and DAC for Pi Zero"
